Commit message: Support Wavefront obj mesh format

File: robots/hsrb4s_obj.urdf (robot description, URDF)
Before this commit: robot hsrb, 45 links, 44 joints
Links:
- link arm_flex_link: geometry collision mesh filename=package://hsr_meshes/meshes/arm_v0/arm_flex.stl; visual mesh filename=package://hsr_meshes/meshes/arm_v0/arm_flex_light.obj
- link arm_lift_link: geometry collision mesh filename=package://hsr_meshes/meshes/arm_v0/shoulder.stl; visual mesh filename=package://hsr_meshes/meshes/arm_v0/shoulder.obj
- link arm_roll_link: geometry collision mesh filename=package://hsr_meshes/meshes/arm_v0/arm_roll.stl; visual mesh filename=package://hsr_meshes/meshes/arm_v0/arm_roll_light.obj
- link base_link: geometry collision mesh filename=package://hsr_meshes/meshes/base_v2/base.stl; visual mesh filename=package://hsr_meshes/meshes/base_v2/base_light.obj
- link base_range_sensor_link: geometry collision mesh filename=package://hsr_meshes/meshes/sensors/laser.stl; visual mesh filename=package://hsr_meshes/meshes/sensors/laser.obj
- link head_l_stereo_camera_link: geometry visual mesh filename=package://hsr_meshes/meshes/sensors/head_camera.obj
- link head_pan_link: geometry collision mesh filename=package://hsr_meshes/meshes/head_v1/head_pan.stl; visual mesh filename=package://hsr_meshes/meshes/head_v1/head_pan.obj
- link head_r_stereo_camera_link: geometry visual mesh filename=package://hsr_meshes/meshes/sensors/head_camera.obj
- link head_rgbd_sensor_link: geometry collision mesh filename=package://hsr_meshes/meshes/sensors/rgbd.stl; visual mesh filename=package://hsr_meshes/meshes/sensors/rgbd_light.obj
- link head_tilt_link: geometry collision mesh filename=package://hsr_meshes/meshes/head_v1/head.stl; collision mesh filename=package://hsr_meshes/meshes/head_v1/tablet.stl
- link torso_lift_link: geometry collision mesh filename=package://hsr_meshes/meshes/torso_v0/torso.stl; visual mesh filename=package://hsr_meshes/meshes/torso_v0/torso_light.obj
- link wrist_flex_link: geometry collision cylinder length=0.04 radius=0.017; visual cylinder length=0.02 radius=0.017
- link wrist_roll_link: geometry collision mesh filename=package://hsr_meshes/meshes/wrist_v0/wrist_roll.stl; visual mesh filename=package://hsr_meshes/meshes/wrist_v0/wrist_roll.obj

File: robots/hsrb4s_obj.urdf.xacro (robot description, xacro)
@@ -43,18 +43,18 @@
     <xacro:property name="robot_name" value="hsrb"/>
     <!-- create robot -->
-    <xacro:hsrb_base prefix="base" robot_namespace="${robot_name}"/>
-    <xacro:hsrb_torso prefix="torso" parent="base_link" mimic_joint="arm_lift_joint">
+    <xacro:hsrb_base prefix="base" robot_namespace="${robot_name}" use_collada="false"/>
+    <xacro:hsrb_torso prefix="torso" parent="base_link" mimic_joint="arm_lift_joint" use_collada="false">
         <origin xyz="0.0 0.0 0.752" rpy="0.0 0.0 0.0"/>
     </xacro:hsrb_torso>
-    <xacro:hsrb_head prefix="head" parent="torso_lift_link">
+    <xacro:hsrb_head prefix="head" parent="torso_lift_link" use_collada="false">
         <origin xyz="0.0 0.0 0.0" rpy="0.0 0.0 0.0"/>
     </xacro:hsrb_head>
-    <xacro:hsrb_arm prefix="arm" parent="base_link">
+    <xacro:hsrb_arm prefix="arm" parent="base_link" use_collada="false">
         <origin xyz="0.0 0.0 0.340" rpy="0.0 0.0 0.0"/>
     </xacro:hsrb_arm>
-    <xacro:hsrb_wrist prefix="wrist" parent="arm_roll_link" robot_namespace="${robot_name}">
+    <xacro:hsrb_wrist prefix="wrist" parent="arm_roll_link" robot_namespace="${robot_name}" use_collada="false">
         <origin xyz="0.0 0.0 0.0" rpy="0.0 0.0 0.0"/>
     </xacro:hsrb_wrist>
-    <xacro:hsrb_hand prefix="hand" parent="wrist_roll_link">
+    <xacro:hsrb_hand prefix="hand" parent="wrist_roll_link" use_collada="false">
         <origin xyz="0.012 0.0 0.1405" rpy="0.0 0.0 ${pi}"/>
     </xacro:hsrb_hand>

File: urdf/arm_v0/arm.urdf.xacro (robot description, xacro)
@@ -29,5 +29,5 @@
     <xacro:include filename="$(find hsr_description)/urdf/arm_v0/arm.gazebo.xacro"/>
     <!-- arm -->
-    <xacro:macro name="hsrb_arm" params="prefix parent *origin">
+    <xacro:macro name="hsrb_arm" params="prefix parent *origin use_collada:=true">
         <joint name="${prefix}_lift_joint" type="prismatic">
             <insert_block name="origin" />
@@ -47,5 +47,10 @@
             <visual>
                 <geometry>
-                    <mesh filename="package://hsr_meshes/meshes/arm_v0/shoulder.dae" />
+                    <xacro:if value="${use_collada}">
+                        <mesh filename="package://hsr_meshes/meshes/arm_v0/shoulder.dae" />
+                    </xacro:if>
+                    <xacro:unless value="${use_collada}">
+                        <mesh filename="package://hsr_meshes/meshes/arm_v0/shoulder.obj" />
+                    </xacro:unless>
                 </geometry>
             </visual>
@@ -73,5 +78,10 @@
             <visual>
                 <geometry>
-                    <mesh filename="package://hsr_meshes/meshes/arm_v0/arm_flex_light.dae" />
+                    <xacro:if value="${use_collada}">
+                        <mesh filename="package://hsr_meshes/meshes/arm_v0/arm_flex_light.dae" />
+                    </xacro:if>
+                    <xacro:unless value="${use_collada}">
+                        <mesh filename="package://hsr_meshes/meshes/arm_v0/arm_flex_light.obj" />
+                    </xacro:unless>
                 </geometry>
             </visual>
@@ -99,5 +109,10 @@
             <visual>
                 <geometry>
-                    <mesh filename="package://hsr_meshes/meshes/arm_v0/arm_roll_light.dae" />
+                    <xacro:if value="${use_collada}">
+                        <mesh filename="package://hsr_meshes/meshes/arm_v0/arm_roll_light.dae" />
+                    </xacro:if>
+                    <xacro:unless value="${use_collada}">
+                        <mesh filename="package://hsr_meshes/meshes/arm_v0/arm_roll_light.obj" />
+                    </xacro:unless>
                 </geometry>
             </visual>

File: urdf/base_v2/base.urdf.xacro (robot description, xacro)
@@ -129,5 +129,5 @@
     </xacro:macro>
     <!-- base -->
-    <xacro:macro name="hsrb_base" params="prefix robot_namespace">
+    <xacro:macro name="hsrb_base" params="prefix robot_namespace use_collada:=true">
         <link name="base_footprint"/>
         <joint name="${prefix}_footprint_joint" type="fixed">
@@ -144,15 +144,30 @@
             <visual>
                 <geometry>
-                    <mesh filename="package://hsr_meshes/meshes/base_v2/base_light.dae" />
-                </geometry>
-            </visual>
-            <visual>
-                <geometry>
-                    <mesh filename="package://hsr_meshes/meshes/base_v2/body_light.dae" />
-                </geometry>
-            </visual>
-            <visual>
-                <geometry>
-                    <mesh filename="package://hsr_meshes/meshes/base_v2/torso_base.dae" />
+                    <xacro:if value="${use_collada}">
+                        <mesh filename="package://hsr_meshes/meshes/base_v2/base_light.dae" />
+                    </xacro:if>
+                    <xacro:unless value="${use_collada}">
+                        <mesh filename="package://hsr_meshes/meshes/base_v2/base_light.obj" />
+                    </xacro:unless>
+                </geometry>
+            </visual>
+            <visual>
+                <geometry>
+                    <xacro:if value="${use_collada}">
+                        <mesh filename="package://hsr_meshes/meshes/base_v2/body_light.dae" />
+                    </xacro:if>
+                    <xacro:unless value="${use_collada}">
+                        <mesh filename="package://hsr_meshes/meshes/base_v2/body_light.obj" />
+                    </xacro:unless>
+                </geometry>
+            </visual>
+            <visual>
+                <geometry>
+                    <xacro:if value="${use_collada}">
+                        <mesh filename="package://hsr_meshes/meshes/base_v2/torso_base.dae" />
+                    </xacro:if>
+                    <xacro:unless value="${use_collada}">
+                        <mesh filename="package://hsr_meshes/meshes/base_v2/torso_base.obj" />
+                    </xacro:unless>
                 </geometry>
             </visual>
@@ -206,5 +221,6 @@
             prefix="${prefix}"
             robot_namespace="${robot_namespace}"
-            parent="${prefix}_link">
+            parent="${prefix}_link"
+            use_collada="${use_collada}">
             <origin xyz="0.1675 0.0 0.1844" rpy="0.0 0.0 0.0" />
         </xacro:laser>

File: urdf/hand_v0/hand.urdf.xacro (robot description, xacro)
@@ -87,5 +87,5 @@
         <xacro:hsrb_gripper_dummy_link name="${prefix}_motor_dummy_link" />
     </xacro:macro>
-    <xacro:macro name="hsrb_hand" params="prefix parent *origin">
+    <xacro:macro name="hsrb_hand" params="prefix parent *origin use_collada:=true">
         <xacro:hsrb_gripper_base prefix="${prefix}" parent="${parent}">
             <insert_block name="origin" />

File: urdf/head_v2/head.urdf.xacro (robot description, xacro)
@@ -32,5 +32,5 @@
     <xacro:include filename="$(find hsr_description)/urdf/sensors/wide_camera.urdf.xacro"/>
     <!-- head -->
-    <xacro:macro name="hsrb_head" params="prefix parent *origin">
+    <xacro:macro name="hsrb_head" params="prefix parent *origin use_collada:=true">
         <joint name="${prefix}_pan_joint" type="revolute">
             <insert_block name="origin" />
@@ -50,5 +50,10 @@
             <visual>
                 <geometry>
-                    <mesh filename="package://hsr_meshes/meshes/head_v1/head_pan.dae" />
+                    <xacro:if value="${use_collada}">
+                        <mesh filename="package://hsr_meshes/meshes/head_v1/head_pan.dae" />
+                    </xacro:if>
+                    <xacro:unless value="${use_collada}">
+                        <mesh filename="package://hsr_meshes/meshes/head_v1/head_pan.obj" />
+                    </xacro:unless>
                 </geometry>
             </visual>
@@ -76,15 +81,30 @@
             <visual>
                 <geometry>
-                    <mesh filename="package://hsr_meshes/meshes/head_v1/head_upper.dae" />
+                    <xacro:if value="${use_collada}">
+                        <mesh filename="package://hsr_meshes/meshes/head_v1/head_upper.dae" />
+                    </xacro:if>
+                    <xacro:unless value="${use_collada}">
+                        <mesh filename="package://hsr_meshes/meshes/head_v1/head_upper.obj" />
+                    </xacro:unless>
                 </geometry>
             </visual>
             <visual>
                 <geometry>
-                    <mesh filename="package://hsr_meshes/meshes/head_v1/head_tilt.dae" />
+                    <xacro:if value="${use_collada}">
+                        <mesh filename="package://hsr_meshes/meshes/head_v1/head_tilt.dae" />
+                    </xacro:if>
+                    <xacro:unless value="${use_collada}">
+                        <mesh filename="package://hsr_meshes/meshes/head_v1/head_tilt.obj" />
+                    </xacro:unless>
                 </geometry>
             </visual>
             <visual>
                 <geometry>
-                    <mesh filename="package://hsr_meshes/meshes/head_v1/tablet_base.dae" />
+                    <xacro:if value="${use_collada}">
+                        <mesh filename="package://hsr_meshes/meshes/head_v1/tablet_base.dae" />
+                    </xacro:if>
+                    <xacro:unless value="${use_collada}">
+                        <mesh filename="package://hsr_meshes/meshes/head_v1/tablet_base.obj" />
+                    </xacro:unless>
                 </geometry>
             </visual>
@@ -101,8 +121,8 @@
         </link>
         <!-- cameras -->
-        <xacro:rgb_sensor prefix="${prefix}_l_stereo" parent="${prefix}_tilt_link" robot_namespace="${robot_name}" baseline="0.00">
+        <xacro:rgb_sensor prefix="${prefix}_l_stereo" parent="${prefix}_tilt_link" robot_namespace="${robot_name}" baseline="0.00" use_collada="${use_collada}">
             <origin xyz="0.02 0.07 0.061" rpy="${-pi/2.0} 0.0 ${-pi/2.0}"/>
         </xacro:rgb_sensor>
-        <xacro:rgb_sensor prefix="${prefix}_r_stereo" parent="${prefix}_tilt_link" robot_namespace="${robot_name}" baseline="0.14">
+        <xacro:rgb_sensor prefix="${prefix}_r_stereo" parent="${prefix}_tilt_link" robot_namespace="${robot_name}" baseline="0.14" use_collada="${use_collada}">
             <origin xyz="0.02 -0.07 0.061" rpy="${-pi/2.0} 0.0 ${-pi/2.0}"/>
         </xacro:rgb_sensor>
@@ -110,5 +130,5 @@
             <origin xyz="0.0195 0.0 0.061" rpy="${-pi/2.0} 0.0 ${-pi/2.0}"/>
         </xacro:wide_camera>
-        <xacro:rgbd_sensor prefix="${prefix}" parent="${prefix}_tilt_link" robot_namespace="${robot_name}" sensor_name="rgbd_sensor">
+        <xacro:rgbd_sensor prefix="${prefix}" parent="${prefix}_tilt_link" robot_namespace="${robot_name}" sensor_name="rgbd_sensor" use_collada="${use_collada}">
             <origin xyz="-0.079796 0.022 0.215172" rpy="${-pi/2.0} 0.0 ${-pi/2.0}"/>
         </xacro:rgbd_sensor>

File: urdf/sensors/laser.urdf.xacro (robot description, xacro)
@@ -28,5 +28,5 @@
     <xacro:include filename="$(find hsr_description)/urdf/sensors/laser.gazebo.xacro"/>
     <!-- range sensor -->
-    <xacro:macro name="laser" params="prefix robot_namespace parent *origin">
+    <xacro:macro name="laser" params="prefix robot_namespace parent *origin use_collada:=true">
         <joint name="${prefix}_range_sensor_joint" type="fixed">
             <insert_block name="origin" />
@@ -37,5 +37,10 @@
             <visual>
                 <geometry>
-                    <mesh filename="package://hsr_meshes/meshes/sensors/laser.dae" />
+                    <xacro:if value="${use_collada}">
+                        <mesh filename="package://hsr_meshes/meshes/sensors/laser.dae" />
+                    </xacro:if>
+                    <xacro:unless value="${use_collada}">
+                        <mesh filename="package://hsr_meshes/meshes/sensors/laser.obj" />
+                    </xacro:unless>
                 </geometry>
             </visual>

File: urdf/sensors/rgb_sensor.urdf.xacro (robot description, xacro)
@@ -27,5 +27,5 @@
 <robot xmlns:xacro="http://ros.org/wiki/xacro">
     <xacro:include filename="$(find hsr_description)/urdf/sensors/rgb_sensor.gazebo.xacro"/>
-    <xacro:macro name="rgb_sensor" params="prefix parent robot_namespace *origin baseline">
+    <xacro:macro name="rgb_sensor" params="prefix parent robot_namespace *origin baseline use_collada:=true">
         <joint name="${prefix}_camera_joint" type="fixed">
             <insert_block name="origin" />
@@ -37,5 +37,10 @@
                 <origin xyz="0 0 0" rpy="0.0 0.0 0.0"/>
                 <geometry>
-                    <mesh filename="package://hsr_meshes/meshes/sensors/head_camera.dae" />
+                    <xacro:if value="${use_collada}">
+                        <mesh filename="package://hsr_meshes/meshes/sensors/head_camera.dae" />
+                    </xacro:if>
+                    <xacro:unless value="${use_collada}">
+                        <mesh filename="package://hsr_meshes/meshes/sensors/head_camera.obj" />
+                    </xacro:unless>
                 </geometry>
             </visual>

File: urdf/sensors/rgbd_sensor.urdf.xacro (robot description, xacro)
@@ -28,5 +28,5 @@
     <xacro:include filename="$(find hsr_description)/urdf/sensors/rgbd_sensor.gazebo.xacro"/>
     <!-- rgbd_sensor -->
-    <xacro:macro name="rgbd_sensor" params="prefix parent robot_namespace sensor_name *origin">
+    <xacro:macro name="rgbd_sensor" params="prefix parent robot_namespace sensor_name *origin use_collada:=true">
         <joint name="${prefix}_${sensor_name}_joint" type="fixed">
             <insert_block name="origin" />
@@ -37,5 +37,10 @@
                 <origin xyz="0 0 0" rpy="0.0 0.0 0.0"/>
                 <geometry>
-                    <mesh filename="package://hsr_meshes/meshes/sensors/rgbd_light.dae" />
+                    <xacro:if value="${use_collada}">
+                        <mesh filename="package://hsr_meshes/meshes/sensors/rgbd_light.dae" />
+                    </xacro:if>
+                    <xacro:unless value="${use_collada}">
+                        <mesh filename="package://hsr_meshes/meshes/sensors/rgbd_light.obj" />
+                    </xacro:unless>
                 </geometry>
             </visual>

File: urdf/torso_v0/torso.urdf.xacro (robot description, xacro)
@@ -28,5 +28,5 @@
     <xacro:include filename="$(find hsr_description)/urdf/torso_v0/torso.gazebo.xacro"/>
     <!-- torso -->
-    <xacro:macro name="hsrb_torso" params="prefix parent mimic_joint *origin">
+    <xacro:macro name="hsrb_torso" params="prefix parent mimic_joint *origin use_collada:=true">
         <joint name="${prefix}_lift_joint" type="prismatic">
             <insert_block name="origin" />
@@ -48,5 +48,10 @@
             <visual>
                 <geometry>
-                    <mesh filename="package://hsr_meshes/meshes/torso_v0/torso_light.dae" />
+                    <xacro:if value="${use_collada}">
+                        <mesh filename="package://hsr_meshes/meshes/torso_v0/torso_light.dae" />
+                    </xacro:if>
+                    <xacro:unless value="${use_collada}">
+                        <mesh filename="package://hsr_meshes/meshes/torso_v0/torso_light.obj" />
+                    </xacro:unless>
                 </geometry>
             </visual>

File: urdf/wrist_v0/wrist.urdf.xacro (robot description, xacro)
@@ -30,5 +30,5 @@
     <xacro:include filename="$(find hsr_description)/urdf/sensors/ft_sensor.urdf.xacro"/>
     <!-- wrist -->
-    <xacro:macro name="hsrb_wrist" params="prefix robot_namespace parent *origin">
+    <xacro:macro name="hsrb_wrist" params="prefix robot_namespace parent *origin use_collada:=true">
         <joint name="${prefix}_flex_joint" type="revolute">
             <origin xyz="0.0 0.0 0.0" rpy="0.0 0.0 0.0" />
@@ -48,5 +48,10 @@
             <visual>
                 <geometry>
-                    <mesh filename="package://hsr_meshes/meshes/wrist_v0/wrist_flex.dae" />
+                    <xacro:if value="${use_collada}">
+                        <mesh filename="package://hsr_meshes/meshes/wrist_v0/wrist_flex.dae" />
+                    </xacro:if>
+                    <xacro:unless value="${use_collada}">
+                        <mesh filename="package://hsr_meshes/meshes/wrist_v0/wrist_flex.obj" />
+                    </xacro:unless>
                 </geometry>
                 <material name="body_sub" />
@@ -83,5 +88,10 @@
             <visual>
                 <geometry>
-                    <mesh filename="package://hsr_meshes/meshes/wrist_v0/wrist_roll.dae" />
+                    <xacro:if value="${use_collada}">
+                        <mesh filename="package://hsr_meshes/meshes/wrist_v0/wrist_roll.dae" />
+                    </xacro:if>
+                    <xacro:unless value="${use_collada}">
+                        <mesh filename="package://hsr_meshes/meshes/wrist_v0/wrist_roll.obj" />
+                    </xacro:unless>
                 </geometry>
             </visual>
