Commit message: Update to use OBJ instead of STL

File: robots/hsrb4s.obj.urdf (robot description, URDF)
Before this commit: robot hsrb, 45 links, 44 joints
Links:
- link hand_l_distal_link: geometry collision mesh filename=package://hsr_meshes/meshes/hand_v0/l_distal.stl; visual mesh filename=package://hsr_meshes/meshes/hand_v0/l_distal.obj
- link hand_palm_link: geometry collision mesh filename=package://hsr_meshes/meshes/hand_v0/palm.stl; visual mesh filename=package://hsr_meshes/meshes/hand_v0/palm.obj
- link hand_r_distal_link: geometry collision mesh filename=package://hsr_meshes/meshes/hand_v0/r_distal.stl; visual mesh filename=package://hsr_meshes/meshes/hand_v0/r_distal.obj
- link hand_r_spring_proximal_link: geometry collision mesh filename=package://hsr_meshes/meshes/hand_v0/r_proximal.stl; visual mesh filename=package://hsr_meshes/meshes/hand_v0/r_proximal.obj

File: robots/hsrb4s.urdf.xacro (robot description, xacro)
@@ -40,8 +40,11 @@
     <xacro:include filename="$(find hsr_description)/urdf/wrist_v0/wrist.urdf.xacro" />
     <xacro:include filename="$(find hsr_description)/urdf/hand_v0/hand.urdf.xacro" />
+    <!-- This switches a format of mesh files for visual property -->
+    <xacro:arg name="use_obj_for_visual" default="false" />
+    <xacro:property name="g_use_obj_for_visual" value="$(arg use_obj_for_visual)"/>
     <!-- constant -->
-    <xacro:property name="robot_name" value="hsrb"/>
+    <xacro:property name="g_robot_name" value="hsrb"/>
     <!-- create robot -->
-    <xacro:hsrb_base prefix="base" robot_namespace="${robot_name}"/>
+    <xacro:hsrb_base prefix="base" robot_namespace="${g_robot_name}"/>
     <xacro:hsrb_torso prefix="torso" parent="base_link" mimic_joint="arm_lift_joint">
         <origin xyz="0.0 0.0 0.752" rpy="0.0 0.0 0.0"/>
@@ -53,5 +56,5 @@
         <origin xyz="0.0 0.0 0.340" rpy="0.0 0.0 0.0"/>
     </xacro:hsrb_arm>
-    <xacro:hsrb_wrist prefix="wrist" parent="arm_roll_link" robot_namespace="${robot_name}">
+    <xacro:hsrb_wrist prefix="wrist" parent="arm_roll_link" robot_namespace="${g_robot_name}">
         <origin xyz="0.0 0.0 0.0" rpy="0.0 0.0 0.0"/>
     </xacro:hsrb_wrist>
@@ -60,9 +63,9 @@
     </xacro:hsrb_hand>
     <gazebo>
-        <plugin name="${robot_name}_ros_control" filename="lib${robot_name}_gazebo_ros_control.so">
-            <robotNamespace>${robot_name}</robotNamespace>
+        <plugin name="${g_robot_name}_ros_control" filename="lib${g_robot_name}_gazebo_ros_control.so">
+            <robotNamespace>${g_robot_name}</robotNamespace>
         </plugin>
-        <plugin name="${robot_name}_p3d_ground_truth" filename="libgazebo_ros_p3d.so">
-            <robotNamespace>${robot_name}</robotNamespace>
+        <plugin name="${g_robot_name}_p3d_ground_truth" filename="libgazebo_ros_p3d.so">
+            <robotNamespace>${g_robot_name}</robotNamespace>
             <bodyName>base_footprint</bodyName>
             <topicName>odom_ground_truth</topicName>

File: urdf/arm_v0/arm.urdf.xacro (robot description, xacro)
@@ -29,5 +29,5 @@
     <xacro:include filename="$(find hsr_description)/urdf/arm_v0/arm.gazebo.xacro"/>
     <!-- arm -->
-    <xacro:macro name="hsrb_arm" params="prefix parent *origin use_collada:=true">
+    <xacro:macro name="hsrb_arm" params="prefix parent *origin">
         <joint name="${prefix}_lift_joint" type="prismatic">
             <insert_block name="origin" />
@@ -47,10 +47,10 @@
             <visual>
                 <geometry>
-                    <xacro:if value="${use_collada}">
+                    <xacro:unless value="${g_use_obj_for_visual}">
                         <mesh filename="package://hsr_meshes/meshes/arm_v0/shoulder.dae" />
+                    </xacro:unless>
+                    <xacro:if value="${g_use_obj_for_visual}">
+                        <mesh filename="package://hsr_meshes/meshes/arm_v0/shoulder.obj" />
                     </xacro:if>
-                    <xacro:unless value="${use_collada}">
-                        <mesh filename="package://hsr_meshes/meshes/arm_v0/shoulder.obj" />
-                    </xacro:unless>
                 </geometry>
             </visual>
@@ -78,10 +78,10 @@
             <visual>
                 <geometry>
-                    <xacro:if value="${use_collada}">
+                    <xacro:unless value="${g_use_obj_for_visual}">
                         <mesh filename="package://hsr_meshes/meshes/arm_v0/arm_flex_light.dae" />
+                    </xacro:unless>
+                    <xacro:if value="${g_use_obj_for_visual}">
+                        <mesh filename="package://hsr_meshes/meshes/arm_v0/arm_flex_light.obj" />
                     </xacro:if>
-                    <xacro:unless value="${use_collada}">
-                        <mesh filename="package://hsr_meshes/meshes/arm_v0/arm_flex_light.obj" />
-                    </xacro:unless>
                 </geometry>
             </visual>
@@ -109,10 +109,10 @@
             <visual>
                 <geometry>
-                    <xacro:if value="${use_collada}">
+                    <xacro:unless value="${g_use_obj_for_visual}">
                         <mesh filename="package://hsr_meshes/meshes/arm_v0/arm_roll_light.dae" />
+                    </xacro:unless>
+                    <xacro:if value="${g_use_obj_for_visual}">
+                        <mesh filename="package://hsr_meshes/meshes/arm_v0/arm_roll_light.obj" />
                     </xacro:if>
-                    <xacro:unless value="${use_collada}">
-                        <mesh filename="package://hsr_meshes/meshes/arm_v0/arm_roll_light.obj" />
-                    </xacro:unless>
                 </geometry>
             </visual>

File: urdf/base_v2/base.urdf.xacro (robot description, xacro)
@@ -129,5 +129,5 @@
     </xacro:macro>
     <!-- base -->
-    <xacro:macro name="hsrb_base" params="prefix robot_namespace use_collada:=true">
+    <xacro:macro name="hsrb_base" params="prefix robot_namespace">
         <link name="base_footprint"/>
         <joint name="${prefix}_footprint_joint" type="fixed">
@@ -144,30 +144,30 @@
             <visual>
                 <geometry>
-                    <xacro:if value="${use_collada}">
+                    <xacro:unless value="${g_use_obj_for_visual}">
                         <mesh filename="package://hsr_meshes/meshes/base_v2/base_light.dae" />
+                    </xacro:unless>
+                    <xacro:if value="${g_use_obj_for_visual}">
+                        <mesh filename="package://hsr_meshes/meshes/base_v2/base_light.obj" />
                     </xacro:if>
-                    <xacro:unless value="${use_collada}">
-                        <mesh filename="package://hsr_meshes/meshes/base_v2/base_light.obj" />
+                </geometry>
+            </visual>
+            <visual>
+                <geometry>
+                    <xacro:unless value="${g_use_obj_for_visual}">
+                        <mesh filename="package://hsr_meshes/meshes/base_v2/body_light.dae" />
                     </xacro:unless>
-                </geometry>
-            </visual>
-            <visual>
-                <geometry>
-                    <xacro:if value="${use_collada}">
-                        <mesh filename="package://hsr_meshes/meshes/base_v2/body_light.dae" />
+                    <xacro:if value="${g_use_obj_for_visual}">
+                        <mesh filename="package://hsr_meshes/meshes/base_v2/body_light.obj" />
                     </xacro:if>
-                    <xacro:unless value="${use_collada}">
-                        <mesh filename="package://hsr_meshes/meshes/base_v2/body_light.obj" />
+                </geometry>
+            </visual>
+            <visual>
+                <geometry>
+                    <xacro:unless value="${g_use_obj_for_visual}">
+                        <mesh filename="package://hsr_meshes/meshes/base_v2/torso_base.dae" />
                     </xacro:unless>
-                </geometry>
-            </visual>
-            <visual>
-                <geometry>
-                    <xacro:if value="${use_collada}">
-                        <mesh filename="package://hsr_meshes/meshes/base_v2/torso_base.dae" />
+                    <xacro:if value="${g_use_obj_for_visual}">
+                        <mesh filename="package://hsr_meshes/meshes/base_v2/torso_base.obj" />
                     </xacro:if>
-                    <xacro:unless value="${use_collada}">
-                        <mesh filename="package://hsr_meshes/meshes/base_v2/torso_base.obj" />
-                    </xacro:unless>
                 </geometry>
             </visual>
@@ -221,6 +221,5 @@
             prefix="${prefix}"
             robot_namespace="${robot_namespace}"
-            parent="${prefix}_link"
-            use_collada="${use_collada}">
+            parent="${prefix}_link">
             <origin xyz="0.1675 0.0 0.1844" rpy="0.0 0.0 0.0" />
         </xacro:laser>

File: urdf/hand_v0/hand.urdf.xacro (robot description, xacro)
@@ -65,5 +65,10 @@
             <visual>
                 <geometry>
-                    <mesh filename="package://hsr_meshes/meshes/hand_v0/palm.stl" />
+                    <xacro:unless value="${g_use_obj_for_visual}">
+                        <mesh filename="package://hsr_meshes/meshes/hand_v0/palm.stl" />
+                    </xacro:unless>
+                    <xacro:if value="${g_use_obj_for_visual}">
+                        <mesh filename="package://hsr_meshes/meshes/hand_v0/palm.obj" />
+                    </xacro:if>
                 </geometry>
                 <material name="body_sub" />
@@ -87,5 +92,5 @@
         <xacro:hsrb_gripper_dummy_link name="${prefix}_motor_dummy_link" />
     </xacro:macro>
-    <xacro:macro name="hsrb_hand" params="prefix parent *origin use_collada:=true">
+    <xacro:macro name="hsrb_hand" params="prefix parent *origin">
         <xacro:hsrb_gripper_base prefix="${prefix}" parent="${parent}">
             <insert_block name="origin" />
@@ -100,5 +105,5 @@
         </xacro:hsrb_finger_without_vacuum>
         <!-- camera -->
-        <xacro:wide_camera prefix="${prefix}" parent="${prefix}_palm_link" robot_namespace="${robot_name}" rpy="${pi/2.0} ${-pi/2.0} 0" >
+        <xacro:wide_camera prefix="${prefix}" parent="${prefix}_palm_link" robot_namespace="${g_robot_name}" rpy="${pi/2.0} ${-pi/2.0} 0" >
             <origin xyz="0.039 0.0 -0.0045" rpy="0.0 0.0 0.0"/>
         </xacro:wide_camera>
@@ -173,5 +178,10 @@
             <visual>
                 <geometry>
-                    <mesh filename="package://hsr_meshes/meshes/hand_v0/l_proximal.stl" />
+                    <xacro:unless value="${g_use_obj_for_visual}">
+                        <mesh filename="package://hsr_meshes/meshes/hand_v0/l_proximal.stl" />
+                    </xacro:unless>
+                    <xacro:if value="${g_use_obj_for_visual}">
+                        <mesh filename="package://hsr_meshes/meshes/hand_v0/l_proximal.obj" />
+                    </xacro:if>
                 </geometry>
                 <material name="body_sub" />
@@ -197,5 +207,10 @@
             <visual>
                 <geometry>
-                    <mesh filename="package://hsr_meshes/meshes/hand_v0/l_distal.stl" />
+                    <xacro:unless value="${g_use_obj_for_visual}">
+                        <mesh filename="package://hsr_meshes/meshes/hand_v0/l_distal.stl" />
+                    </xacro:unless>
+                    <xacro:if value="${g_use_obj_for_visual}">
+                        <mesh filename="package://hsr_meshes/meshes/hand_v0/l_distal.obj" />
+                    </xacro:if>
                 </geometry>
                 <material name="body_sub" />
@@ -251,5 +266,10 @@
             <visual>
                 <geometry>
-                    <mesh filename="package://hsr_meshes/meshes/hand_v0/r_proximal.stl" />
+                    <xacro:unless value="${g_use_obj_for_visual}">
+                        <mesh filename="package://hsr_meshes/meshes/hand_v0/r_proximal.stl" />
+                    </xacro:unless>
+                    <xacro:if value="${g_use_obj_for_visual}">
+                        <mesh filename="package://hsr_meshes/meshes/hand_v0/r_proximal.obj" />
+                    </xacro:if>
                 </geometry>
                 <material name="body_sub" />
@@ -275,5 +295,10 @@
             <visual>
                 <geometry>
-                    <mesh filename="package://hsr_meshes/meshes/hand_v0/r_distal.stl" />
+                    <xacro:unless value="${g_use_obj_for_visual}">
+                        <mesh filename="package://hsr_meshes/meshes/hand_v0/r_distal.stl" />
+                    </xacro:unless>
+                    <xacro:if value="${g_use_obj_for_visual}">
+                        <mesh filename="package://hsr_meshes/meshes/hand_v0/r_distal.obj" />
+                    </xacro:if>
                 </geometry>
                 <material name="body_sub" />

File: urdf/head_v2/head.urdf.xacro (robot description, xacro)
@@ -32,5 +32,5 @@
     <xacro:include filename="$(find hsr_description)/urdf/sensors/wide_camera.urdf.xacro"/>
     <!-- head -->
-    <xacro:macro name="hsrb_head" params="prefix parent *origin use_collada:=true">
+    <xacro:macro name="hsrb_head" params="prefix parent *origin">
         <joint name="${prefix}_pan_joint" type="revolute">
             <insert_block name="origin" />
@@ -50,10 +50,10 @@
             <visual>
                 <geometry>
-                    <xacro:if value="${use_collada}">
+                    <xacro:unless value="${g_use_obj_for_visual}">
                         <mesh filename="package://hsr_meshes/meshes/head_v1/head_pan.dae" />
+                    </xacro:unless>
+                    <xacro:if value="${g_use_obj_for_visual}">
+                        <mesh filename="package://hsr_meshes/meshes/head_v1/head_pan.obj" />
                     </xacro:if>
-                    <xacro:unless value="${use_collada}">
-                        <mesh filename="package://hsr_meshes/meshes/head_v1/head_pan.obj" />
-                    </xacro:unless>
                 </geometry>
             </visual>
@@ -81,30 +81,30 @@
             <visual>
                 <geometry>
-                    <xacro:if value="${use_collada}">
+                    <xacro:unless value="${g_use_obj_for_visual}">
                         <mesh filename="package://hsr_meshes/meshes/head_v1/head_upper.dae" />
+                    </xacro:unless>
+                    <xacro:if value="${g_use_obj_for_visual}">
+                        <mesh filename="package://hsr_meshes/meshes/head_v1/head_upper.obj" />
                     </xacro:if>
-                    <xacro:unless value="${use_collada}">
-                        <mesh filename="package://hsr_meshes/meshes/head_v1/head_upper.obj" />
-                    </xacro:unless>
                 </geometry>
             </visual>
             <visual>
                 <geometry>
-                    <xacro:if value="${use_collada}">
+                    <xacro:unless value="${g_use_obj_for_visual}">
                         <mesh filename="package://hsr_meshes/meshes/head_v1/head_tilt.dae" />
+                    </xacro:unless>
+                    <xacro:if value="${g_use_obj_for_visual}">
+                        <mesh filename="package://hsr_meshes/meshes/head_v1/head_tilt.obj" />
                     </xacro:if>
-                    <xacro:unless value="${use_collada}">
-                        <mesh filename="package://hsr_meshes/meshes/head_v1/head_tilt.obj" />
-                    </xacro:unless>
                 </geometry>
             </visual>
             <visual>
                 <geometry>
-                    <xacro:if value="${use_collada}">
+                    <xacro:unless value="${g_use_obj_for_visual}">
                         <mesh filename="package://hsr_meshes/meshes/head_v1/tablet_base.dae" />
+                    </xacro:unless>
+                    <xacro:if value="${g_use_obj_for_visual}">
+                        <mesh filename="package://hsr_meshes/meshes/head_v1/tablet_base.obj" />
                     </xacro:if>
-                    <xacro:unless value="${use_collada}">
-                        <mesh filename="package://hsr_meshes/meshes/head_v1/tablet_base.obj" />
-                    </xacro:unless>
                 </geometry>
             </visual>
@@ -121,14 +121,14 @@
         </link>
         <!-- cameras -->
-        <xacro:rgb_sensor prefix="${prefix}_l_stereo" parent="${prefix}_tilt_link" robot_namespace="${robot_name}" baseline="0.00" use_collada="${use_collada}">
+        <xacro:rgb_sensor prefix="${prefix}_l_stereo" parent="${prefix}_tilt_link" robot_namespace="${g_robot_name}" baseline="0.00">
             <origin xyz="0.02 0.07 0.061" rpy="${-pi/2.0} 0.0 ${-pi/2.0}"/>
         </xacro:rgb_sensor>
-        <xacro:rgb_sensor prefix="${prefix}_r_stereo" parent="${prefix}_tilt_link" robot_namespace="${robot_name}" baseline="0.14" use_collada="${use_collada}">
+        <xacro:rgb_sensor prefix="${prefix}_r_stereo" parent="${prefix}_tilt_link" robot_namespace="${g_robot_name}" baseline="0.14">
             <origin xyz="0.02 -0.07 0.061" rpy="${-pi/2.0} 0.0 ${-pi/2.0}"/>
         </xacro:rgb_sensor>
-        <xacro:wide_camera prefix="${prefix}_center" parent="${prefix}_tilt_link" robot_namespace="${robot_name}" rpy="${pi/2.0} ${-pi/2.0} 0.0" >
+        <xacro:wide_camera prefix="${prefix}_center" parent="${prefix}_tilt_link" robot_namespace="${g_robot_name}" rpy="${pi/2.0} ${-pi/2.0} 0.0" >
             <origin xyz="0.0195 0.0 0.061" rpy="${-pi/2.0} 0.0 ${-pi/2.0}"/>
         </xacro:wide_camera>
-        <xacro:rgbd_sensor prefix="${prefix}" parent="${prefix}_tilt_link" robot_namespace="${robot_name}" sensor_name="rgbd_sensor" use_collada="${use_collada}">
+        <xacro:rgbd_sensor prefix="${prefix}" parent="${prefix}_tilt_link" robot_namespace="${g_robot_name}" sensor_name="rgbd_sensor">
             <origin xyz="-0.079796 0.022 0.215172" rpy="${-pi/2.0} 0.0 ${-pi/2.0}"/>
         </xacro:rgbd_sensor>

File: urdf/materials.urdf.xacro (robot description, xacro)
@@ -30,5 +30,5 @@
   </material>
   <material name="body_sub">
-    <color rgba="0.33 0.33 0.33 1.0"/>
+    <color rgba="0.3333 0.3333 0.3333 1.0"/>
   </material>
   <material name="wheel">

File: urdf/sensors/laser.urdf.xacro (robot description, xacro)
@@ -28,5 +28,5 @@
     <xacro:include filename="$(find hsr_description)/urdf/sensors/laser.gazebo.xacro"/>
     <!-- range sensor -->
-    <xacro:macro name="laser" params="prefix robot_namespace parent *origin use_collada:=true">
+    <xacro:macro name="laser" params="prefix robot_namespace parent *origin">
         <joint name="${prefix}_range_sensor_joint" type="fixed">
             <insert_block name="origin" />
@@ -37,10 +37,10 @@
             <visual>
                 <geometry>
-                    <xacro:if value="${use_collada}">
+                    <xacro:unless value="${g_use_obj_for_visual}">
                         <mesh filename="package://hsr_meshes/meshes/sensors/laser.dae" />
+                    </xacro:unless>
+                    <xacro:if value="${g_use_obj_for_visual}">
+                        <mesh filename="package://hsr_meshes/meshes/sensors/laser.obj" />
                     </xacro:if>
-                    <xacro:unless value="${use_collada}">
-                        <mesh filename="package://hsr_meshes/meshes/sensors/laser.obj" />
-                    </xacro:unless>
                 </geometry>
             </visual>

File: urdf/sensors/rgb_sensor.urdf.xacro (robot description, xacro)
@@ -27,5 +27,5 @@
 <robot xmlns:xacro="http://ros.org/wiki/xacro">
     <xacro:include filename="$(find hsr_description)/urdf/sensors/rgb_sensor.gazebo.xacro"/>
-    <xacro:macro name="rgb_sensor" params="prefix parent robot_namespace *origin baseline use_collada:=true">
+    <xacro:macro name="rgb_sensor" params="prefix parent robot_namespace *origin baseline">
         <joint name="${prefix}_camera_joint" type="fixed">
             <insert_block name="origin" />
@@ -37,9 +37,9 @@
                 <origin xyz="0 0 0" rpy="0.0 0.0 0.0"/>
                 <geometry>
-                    <xacro:if value="${use_collada}">
+                    <xacro:if value="${g_use_obj_for_visual}">
+                        <mesh filename="package://hsr_meshes/meshes/sensors/head_camera.obj" />
+                    </xacro:if>
+                    <xacro:unless value="${g_use_obj_for_visual}">
                         <mesh filename="package://hsr_meshes/meshes/sensors/head_camera.dae" />
-                    </xacro:if>
-                    <xacro:unless value="${use_collada}">
-                        <mesh filename="package://hsr_meshes/meshes/sensors/head_camera.obj" />
                     </xacro:unless>
                 </geometry>

File: urdf/sensors/rgbd_sensor.urdf.xacro (robot description, xacro)
@@ -28,5 +28,5 @@
     <xacro:include filename="$(find hsr_description)/urdf/sensors/rgbd_sensor.gazebo.xacro"/>
     <!-- rgbd_sensor -->
-    <xacro:macro name="rgbd_sensor" params="prefix parent robot_namespace sensor_name *origin use_collada:=true">
+    <xacro:macro name="rgbd_sensor" params="prefix parent robot_namespace sensor_name *origin">
         <joint name="${prefix}_${sensor_name}_joint" type="fixed">
             <insert_block name="origin" />
@@ -37,10 +37,10 @@
                 <origin xyz="0 0 0" rpy="0.0 0.0 0.0"/>
                 <geometry>
-                    <xacro:if value="${use_collada}">
+                    <xacro:unless value="${g_use_obj_for_visual}">
                         <mesh filename="package://hsr_meshes/meshes/sensors/rgbd_light.dae" />
+                    </xacro:unless>
+                    <xacro:if value="${g_use_obj_for_visual}">
+                        <mesh filename="package://hsr_meshes/meshes/sensors/rgbd_light.obj" />
                     </xacro:if>
-                    <xacro:unless value="${use_collada}">
-                        <mesh filename="package://hsr_meshes/meshes/sensors/rgbd_light.obj" />
-                    </xacro:unless>
                 </geometry>
             </visual>
