Commit message: Update to use OBJ instead of STL

File: urdf/torso_v0/torso.urdf.xacro (robot description, xacro)
@@ -28,5 +28,5 @@
     <xacro:include filename="$(find hsr_description)/urdf/torso_v0/torso.gazebo.xacro"/>
     <!-- torso -->
-    <xacro:macro name="hsrb_torso" params="prefix parent mimic_joint *origin use_collada:=true">
+    <xacro:macro name="hsrb_torso" params="prefix parent mimic_joint *origin">
         <joint name="${prefix}_lift_joint" type="prismatic">
             <insert_block name="origin" />
@@ -48,10 +48,10 @@
             <visual>
                 <geometry>
-                    <xacro:if value="${use_collada}">
+                    <xacro:unless value="${g_use_obj_for_visual}">
                         <mesh filename="package://hsr_meshes/meshes/torso_v0/torso_light.dae" />
+                    </xacro:unless>
+                    <xacro:if value="${g_use_obj_for_visual}">
+                        <mesh filename="package://hsr_meshes/meshes/torso_v0/torso_light.obj" />
                     </xacro:if>
-                    <xacro:unless value="${use_collada}">
-                        <mesh filename="package://hsr_meshes/meshes/torso_v0/torso_light.obj" />
-                    </xacro:unless>
                 </geometry>
             </visual>

File: urdf/wrist_v0/wrist.urdf.xacro (robot description, xacro)
@@ -30,5 +30,5 @@
     <xacro:include filename="$(find hsr_description)/urdf/sensors/ft_sensor.urdf.xacro"/>
     <!-- wrist -->
-    <xacro:macro name="hsrb_wrist" params="prefix robot_namespace parent *origin use_collada:=true">
+    <xacro:macro name="hsrb_wrist" params="prefix robot_namespace parent *origin">
         <joint name="${prefix}_flex_joint" type="revolute">
             <origin xyz="0.0 0.0 0.0" rpy="0.0 0.0 0.0" />
@@ -48,10 +48,10 @@
             <visual>
                 <geometry>
-                    <xacro:if value="${use_collada}">
+                    <xacro:unless value="${g_use_obj_for_visual}">
                         <mesh filename="package://hsr_meshes/meshes/wrist_v0/wrist_flex.dae" />
+                    </xacro:unless>
+                    <xacro:if value="${g_use_obj_for_visual}">
+                        <mesh filename="package://hsr_meshes/meshes/wrist_v0/wrist_flex.obj" />
                     </xacro:if>
-                    <xacro:unless value="${use_collada}">
-                        <mesh filename="package://hsr_meshes/meshes/wrist_v0/wrist_flex.obj" />
-                    </xacro:unless>
                 </geometry>
                 <material name="body_sub" />
@@ -88,10 +88,10 @@
             <visual>
                 <geometry>
-                    <xacro:if value="${use_collada}">
+                    <xacro:unless value="${g_use_obj_for_visual}">
                         <mesh filename="package://hsr_meshes/meshes/wrist_v0/wrist_roll.dae" />
+                    </xacro:unless>
+                    <xacro:if value="${g_use_obj_for_visual}">
+                        <mesh filename="package://hsr_meshes/meshes/wrist_v0/wrist_roll.obj" />
                     </xacro:if>
-                    <xacro:unless value="${use_collada}">
-                        <mesh filename="package://hsr_meshes/meshes/wrist_v0/wrist_roll.obj" />
-                    </xacro:unless>
                 </geometry>
             </visual>

Commit message: Update URDF robot files

File: robots/hsrb4s.obj.urdf (robot description, URDF)
Before this commit: robot hsrb, 45 links, 44 joints
Links:
- link hand_l_spring_proximal_link: geometry collision mesh filename=package://hsr_meshes/meshes/hand_v0/l_proximal.stl; visual mesh filename=package://hsr_meshes/meshes/hand_v0/l_proximal.obj

Commit message: Fix collision geometry to also use .obj instead of .stl

File: robots/hsrb4s.obj.urdf (robot description, URDF)
Before this commit: robot hsrb, 45 links, 44 joints
Links:
- link arm_flex_link: geometry collision mesh filename=package://hsr_meshes/meshes/arm_v0/arm_flex.obj; visual mesh filename=package://hsr_meshes/meshes/arm_v0/arm_flex_light.obj
- link arm_lift_link: geometry collision mesh filename=package://hsr_meshes/meshes/arm_v0/shoulder.obj; visual mesh filename=package://hsr_meshes/meshes/arm_v0/shoulder.obj
- link arm_roll_link: geometry collision mesh filename=package://hsr_meshes/meshes/arm_v0/arm_roll.obj; visual mesh filename=package://hsr_meshes/meshes/arm_v0/arm_roll_light.obj
- link base_link: geometry collision mesh filename=package://hsr_meshes/meshes/base_v2/base.obj; visual mesh filename=package://hsr_meshes/meshes/base_v2/base_light.obj
- link base_range_sensor_link: geometry collision mesh filename=package://hsr_meshes/meshes/sensors/laser.obj; visual mesh filename=package://hsr_meshes/meshes/sensors/laser.obj
- link hand_l_distal_link: geometry collision mesh filename=package://hsr_meshes/meshes/hand_v0/l_distal.obj; visual mesh filename=package://hsr_meshes/meshes/hand_v0/l_distal.obj
- link hand_l_spring_proximal_link: geometry collision mesh filename=package://hsr_meshes/meshes/hand_v0/l_proximal.obj; visual mesh filename=package://hsr_meshes/meshes/hand_v0/l_proximal.obj
- link hand_palm_link: geometry collision mesh filename=package://hsr_meshes/meshes/hand_v0/palm.obj; visual mesh filename=package://hsr_meshes/meshes/hand_v0/palm.obj
- link hand_r_distal_link: geometry collision mesh filename=package://hsr_meshes/meshes/hand_v0/r_distal.obj; visual mesh filename=package://hsr_meshes/meshes/hand_v0/r_distal.obj
- link hand_r_spring_proximal_link: geometry collision mesh filename=package://hsr_meshes/meshes/hand_v0/r_proximal.obj; visual mesh filename=package://hsr_meshes/meshes/hand_v0/r_proximal.obj
- link head_pan_link: geometry collision mesh filename=package://hsr_meshes/meshes/head_v1/head_pan.obj; visual mesh filename=package://hsr_meshes/meshes/head_v1/head_pan.obj
- link head_rgbd_sensor_link: geometry collision mesh filename=package://hsr_meshes/meshes/sensors/rgbd.obj; visual mesh filename=package://hsr_meshes/meshes/sensors/rgbd_light.obj
- link head_tilt_link: geometry collision mesh filename=package://hsr_meshes/meshes/head_v1/head.obj; collision mesh filename=package://hsr_meshes/meshes/head_v1/tablet.obj
- link torso_lift_link: geometry collision mesh filename=package://hsr_meshes/meshes/torso_v0/torso.obj; visual mesh filename=package://hsr_meshes/meshes/torso_v0/torso_light.obj
- link wrist_roll_link: geometry collision mesh filename=package://hsr_meshes/meshes/wrist_v0/wrist_roll.obj; visual mesh filename=package://hsr_meshes/meshes/wrist_v0/wrist_roll.obj

Commit message: Use OBJ format for visual and collision element

File: robots/hsrb4s.obj.urdf (robot description, URDF)
Before this commit: robot hsrb, 45 links, 44 joints
Links:
- link arm_flex_link: geometry collision mesh filename=package://hsr_meshes/meshes/arm_v0/arm_flex.collision.obj; visual mesh filename=package://hsr_meshes/meshes/arm_v0/arm_flex_light.obj
- link arm_lift_link: geometry collision mesh filename=package://hsr_meshes/meshes/arm_v0/shoulder.collision.obj; visual mesh filename=package://hsr_meshes/meshes/arm_v0/shoulder.obj
- link arm_roll_link: geometry collision mesh filename=package://hsr_meshes/meshes/arm_v0/arm_roll.collision.obj; visual mesh filename=package://hsr_meshes/meshes/arm_v0/arm_roll_light.obj
- link base_link: geometry collision mesh filename=package://hsr_meshes/meshes/base_v2/base.collision.obj; visual mesh filename=package://hsr_meshes/meshes/base_v2/base_light.obj
- link base_range_sensor_link: geometry collision mesh filename=package://hsr_meshes/meshes/sensors/laser.obj; visual mesh filename=package://hsr_meshes/meshes/sensors/laser.obj
- link hand_l_distal_link: geometry collision mesh filename=package://hsr_meshes/meshes/hand_v0/l_distal.obj; visual mesh filename=package://hsr_meshes/meshes/hand_v0/l_distal.obj
- link hand_l_spring_proximal_link: geometry collision mesh filename=package://hsr_meshes/meshes/hand_v0/l_proximal.obj; visual mesh filename=package://hsr_meshes/meshes/hand_v0/l_proximal.obj
- link hand_palm_link: geometry collision mesh filename=package://hsr_meshes/meshes/hand_v0/palm.obj; visual mesh filename=package://hsr_meshes/meshes/hand_v0/palm.obj
- link hand_r_distal_link: geometry collision mesh filename=package://hsr_meshes/meshes/hand_v0/r_distal.obj; visual mesh filename=package://hsr_meshes/meshes/hand_v0/r_distal.obj
- link hand_r_spring_proximal_link: geometry collision mesh filename=package://hsr_meshes/meshes/hand_v0/r_proximal.obj; visual mesh filename=package://hsr_meshes/meshes/hand_v0/r_proximal.obj
- link head_pan_link: geometry collision mesh filename=package://hsr_meshes/meshes/head_v1/head_pan.obj; visual mesh filename=package://hsr_meshes/meshes/head_v1/head_pan.obj
- link head_rgbd_sensor_link: geometry collision mesh filename=package://hsr_meshes/meshes/sensors/rgbd.obj; visual mesh filename=package://hsr_meshes/meshes/sensors/rgbd_light.obj
- link head_tilt_link: geometry collision mesh filename=package://hsr_meshes/meshes/head_v1/head.obj; collision mesh filename=package://hsr_meshes/meshes/head_v1/tablet.obj
- link torso_lift_link: geometry collision mesh filename=package://hsr_meshes/meshes/torso_v0/torso.collision.obj; visual mesh filename=package://hsr_meshes/meshes/torso_v0/torso_light.obj
- link wrist_roll_link: geometry collision mesh filename=package://hsr_meshes/meshes/wrist_v0/wrist_roll.collision.o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; visual mesh filename=package://hsr_meshes/meshes/wrist_v0/wrist_roll.obj

File: robots/hsrb4s.urdf (robot description, URDF)
Before this commit: robot hsrb, 45 links, 44 joints
Links:
- link torso_lift_link: geometry collision mesh filename=package://hsr_meshes/meshes/torso_v0/torso.std; visual mesh filename=package://hsr_meshes/meshes/torso_v0/torso_light.dae

File: robots/hsrb4s.urdf.xacro (robot description, xacro)
@@ -42,5 +42,7 @@
     <!-- This switches a format of mesh files for visual property -->
     <xacro:arg name="use_obj_for_visual" default="false" />
+    <xacro:arg name="use_obj_for_collision" default="false" />
     <xacro:property name="g_use_obj_for_visual" value="$(arg use_obj_for_visual)"/>
+    <xacro:property name="g_use_obj_for_collision" value="$(arg use_obj_for_collision)"/>
     <!-- constant -->
     <xacro:property name="g_robot_name" value="hsrb"/>

File: urdf/arm_v0/arm.urdf.xacro (robot description, xacro)
@@ -57,5 +57,10 @@
             <collision>
                 <geometry>
-                    <mesh filename="package://hsr_meshes/meshes/arm_v0/shoulder.stl" />
+                    <xacro:unless value="${g_use_obj_for_collision}">
+                        <mesh filename="package://hsr_meshes/meshes/arm_v0/shoulder.stl" />
+                    </xacro:unless>
+                    <xacro:if value="${g_use_obj_for_collision}">
+                        <mesh filename="package://hsr_meshes/meshes/arm_v0/shoulder.collision.obj" />
+                    </xacro:if>
                 </geometry>
             </collision>
@@ -72,7 +77,6 @@
             <inertial>
                 <mass value="1.339295"/>
-                <origin xyz="0.000632 0.006404 0.118529"/>
-                <inertia ixx="7.528" ixy="-0.000020284207" ixz="-0.000022947194"
-                    iyy="0.007102" iyz="-0.000091796075" izz="0.001552"/>
+                <origin xyz="-0.000459 0.006583 0.106069"/>
+                <inertia ixx="0.00889053" ixy="0.0" ixz="0.0" iyy="0.00825549" iyz="0.0" izz="0.00190511"/>
             </inertial>
             <visual>
@@ -88,5 +92,10 @@
             <collision>
                 <geometry>
-                    <mesh filename="package://hsr_meshes/meshes/arm_v0/arm_flex.stl" />
+                    <xacro:unless value="${g_use_obj_for_collision}">
+                        <mesh filename="package://hsr_meshes/meshes/arm_v0/arm_flex.stl" />
+                    </xacro:unless>
+                    <xacro:if value="${g_use_obj_for_collision}">
+                        <mesh filename="package://hsr_meshes/meshes/arm_v0/arm_flex.collision.obj" />
+                    </xacro:if>
                 </geometry>
             </collision>
@@ -119,5 +128,10 @@
             <collision>
                 <geometry>
-                    <mesh filename="package://hsr_meshes/meshes/arm_v0/arm_roll.stl" />
+                    <xacro:unless value="${g_use_obj_for_collision}">
+                        <mesh filename="package://hsr_meshes/meshes/arm_v0/arm_roll.stl" />
+                    </xacro:unless>
+                    <xacro:if value="${g_use_obj_for_collision}">
+                        <mesh filename="package://hsr_meshes/meshes/arm_v0/arm_roll.collision.obj" />
+                    </xacro:if>
                 </geometry>
             </collision>

File: urdf/base_v2/base.urdf.xacro (robot description, xacro)
@@ -174,6 +174,11 @@
             <collision>
                 <geometry>
-                    <mesh filename="package://hsr_meshes/meshes/base_v2/base.stl" />
-                </geometry>
+                    <xacro:unless value="${g_use_obj_for_collision}">
+                        <mesh filename="package://hsr_meshes/meshes/base_v2/base.stl" />
+	            </xacro:unless>
+		    <xacro:if value="${g_use_obj_for_collision}">
+			<mesh filename="package://hsr_meshes/meshes/base_v2/base.collision.obj" />
+                    </xacro:if>
+		</geometry>
             </collision>
         </link>

File: urdf/hand_v0/hand.urdf.xacro (robot description, xacro)
@@ -76,5 +76,10 @@
             <collision>
                 <geometry>
-                    <mesh filename="package://hsr_meshes/meshes/hand_v0/palm.stl" />
+                    <xacro:unless value="${g_use_obj_for_collision}">
+                        <mesh filename="package://hsr_meshes/meshes/hand_v0/palm.stl" />
+                    </xacro:unless>
+                    <xacro:if value="${g_use_obj_for_collision}">
+                        <mesh filename="package://hsr_meshes/meshes/hand_v0/palm.obj" />
+                    </xacro:if>
                 </geometry>
             </collision>
@@ -189,5 +194,10 @@
             <collision>
                 <geometry>
-                    <mesh filename="package://hsr_meshes/meshes/hand_v0/l_proximal.stl" />
+                    <xacro:unless value="${g_use_obj_for_collision}">
+                        <mesh filename="package://hsr_meshes/meshes/hand_v0/l_proximal.stl" />
+                    </xacro:unless>
+                    <xacro:if value="${g_use_obj_for_collision}">
+                        <mesh filename="package://hsr_meshes/meshes/hand_v0/l_proximal.obj" />
+                    </xacro:if>
                 </geometry>
             </collision>
@@ -202,6 +212,6 @@
                 <origin xyz="0.011116 0.005679 0.017532"/>
                 <inertia
-                    ixx="0.000004451952" ixy="-0.000000617574" ixz="0.000000503765"
-                    iyy="0.000000503765" iyz="-0.000000435048" izz="0.000004456764"/>
+                    ixx="0.000004451952" ixy="0.0" ixz="0.0"
+                    iyy="0.000000503765" iyz="0.0" izz="0.000004456764"/>
             </inertial>
             <visual>
@@ -218,5 +228,10 @@
             <collision>
                 <geometry>
-                    <mesh filename="package://hsr_meshes/meshes/hand_v0/l_distal.stl" />
+                    <xacro:unless value="${g_use_obj_for_collision}">
+                        <mesh filename="package://hsr_meshes/meshes/hand_v0/l_distal.stl" />
+                    </xacro:unless>
+                    <xacro:if value="${g_use_obj_for_collision}">
+                        <mesh filename="package://hsr_meshes/meshes/hand_v0/l_distal.obj" />
+                    </xacro:if>
                 </geometry>
             </collision>
@@ -277,5 +292,10 @@
             <collision>
                 <geometry>
-                    <mesh filename="package://hsr_meshes/meshes/hand_v0/r_proximal.stl" />
+                    <xacro:unless value="${g_use_obj_for_collision}">
+                        <mesh filename="package://hsr_meshes/meshes/hand_v0/r_proximal.stl" />
+                    </xacro:unless>
+                    <xacro:if value="${g_use_obj_for_collision}">
+                        <mesh filename="package://hsr_meshes/meshes/hand_v0/r_proximal.obj" />
+                    </xacro:if>
                 </geometry>
             </collision>
@@ -306,5 +326,10 @@
             <collision>
                 <geometry>
-                    <mesh filename="package://hsr_meshes/meshes/hand_v0/r_distal.stl" />
+                    <xacro:unless value="${g_use_obj_for_collision}">
+                        <mesh filename="package://hsr_meshes/meshes/hand_v0/r_distal.stl" />
+                    </xacro:unless>
+                    <xacro:if value="${g_use_obj_for_collision}">
+                        <mesh filename="package://hsr_meshes/meshes/hand_v0/r_distal.obj" />
+                    </xacro:if>
                 </geometry>
             </collision>

File: urdf/head_v2/head.urdf.xacro (robot description, xacro)
@@ -60,5 +60,10 @@
             <collision>
                 <geometry>
-                    <mesh filename="package://hsr_meshes/meshes/head_v1/head_pan.stl" />
+                    <xacro:unless value="${g_use_obj_for_collision}">
+                        <mesh filename="package://hsr_meshes/meshes/head_v1/head_pan.stl" />
+                    </xacro:unless>
+                    <xacro:if value="${g_use_obj_for_collision}">
+                        <mesh filename="package://hsr_meshes/meshes/head_v1/head_pan.obj" />
+                    </xacro:if>
                 </geometry>
             </collision>
@@ -111,10 +116,20 @@
             <collision>
                 <geometry>
-                    <mesh filename="package://hsr_meshes/meshes/head_v1/head.stl" />
+                    <xacro:unless value="${g_use_obj_for_collision}">
+                        <mesh filename="package://hsr_meshes/meshes/head_v1/head.stl" />
+                    </xacro:unless>
+                    <xacro:if value="${g_use_obj_for_collision}">
+                        <mesh filename="package://hsr_meshes/meshes/head_v1/head.obj" />
+                    </xacro:if>
                 </geometry>
             </collision>
             <collision>
                 <geometry>
-                    <mesh filename="package://hsr_meshes/meshes/head_v1/tablet.stl" />
+                    <xacro:unless value="${g_use_obj_for_collision}">
+                        <mesh filename="package://hsr_meshes/meshes/head_v1/tablet.stl" />
+                    </xacro:unless>
+                    <xacro:if value="${g_use_obj_for_collision}">
+                        <mesh filename="package://hsr_meshes/meshes/head_v1/tablet.obj" />
+                    </xacro:if>
                 </geometry>
             </collision>

File: urdf/sensors/laser.urdf.xacro (robot description, xacro)
@@ -47,5 +47,10 @@
             <collision>
                 <geometry>
-                    <mesh filename="package://hsr_meshes/meshes/sensors/laser.stl" />
+                    <xacro:unless value="${g_use_obj_for_collision}">
+                        <mesh filename="package://hsr_meshes/meshes/sensors/laser.stl" />
+                    </xacro:unless>
+                    <xacro:if value="${g_use_obj_for_collision}">
+                        <mesh filename="package://hsr_meshes/meshes/sensors/laser.obj" />
+                    </xacro:if>
                 </geometry>
             </collision>

File: urdf/sensors/rgbd_sensor.urdf.xacro (robot description, xacro)
@@ -46,7 +46,12 @@
             </visual>
             <collision>
-                <origin xyz="0 0 0" rpy="0.0 0.0 0.0"/>
-                <geometry>
-                    <mesh filename="package://hsr_meshes/meshes/sensors/rgbd.stl" />
+               <origin xyz="0 0 0" rpy="0.0 0.0 0.0"/>
+               <geometry>
+                  <xacro:unless value="${g_use_obj_for_collision}">
+                     <mesh filename="package://hsr_meshes/meshes/sensors/rgbd.stl" />
+                  </xacro:unless>
+                  <xacro:if value="${g_use_obj_for_collision}">
+                     <mesh filename="package://hsr_meshes/meshes/sensors/rgbd.obj" />
+                  </xacro:if>
                 </geometry>
             </collision>

File: urdf/torso_v0/torso.urdf.xacro (robot description, xacro)
@@ -58,5 +58,10 @@
             <collision>
                 <geometry>
-                    <mesh filename="package://hsr_meshes/meshes/torso_v0/torso.stl" />
+                    <xacro:unless value="${g_use_obj_for_collision}">
+                        <mesh filename="package://hsr_meshes/meshes/torso_v0/torso.std" />
+                    </xacro:unless>
+                    <xacro:if value="${g_use_obj_for_collision}">
+                        <mesh filename="package://hsr_meshes/meshes/torso_v0/torso.collision.obj" />
+                    </xacro:if>
                 </geometry>
             </collision>

File: urdf/wrist_v0/wrist.urdf.xacro (robot description, xacro)
@@ -84,13 +84,13 @@
                 <origin xyz="-0.001416 -0.001547 0.081689"/>
                 <inertia ixx="0.000805633819" ixy="-0.000014431758" ixz="0.000028204659"
-                    iyy="0.000768077165" iyz="0.000022460226" izz="0.000453406611"/>
+                         iyy="0.000768077165" iyz="0.000022460226" izz="0.000453406611"/>
             </inertial>
             <visual>
                 <geometry>
                     <xacro:unless value="${g_use_obj_for_visual}">
-                        <mesh filename="package://hsr_meshes/meshes/wrist_v0/wrist_roll.dae" />
+                       <mesh filename="package://hsr_meshes/meshes/wrist_v0/wrist_roll.dae" />
                     </xacro:unless>
                     <xacro:if value="${g_use_obj_for_visual}">
-                        <mesh filename="package://hsr_meshes/meshes/wrist_v0/wrist_roll.obj" />
+                       <mesh filename="package://hsr_meshes/meshes/wrist_v0/wrist_roll.obj" />
                     </xacro:if>
                 </geometry>
@@ -98,5 +98,10 @@
             <collision>
                 <geometry>
-                    <mesh filename="package://hsr_meshes/meshes/wrist_v0/wrist_roll.stl" />
+                    <xacro:unless value="${g_use_obj_for_collision}">
+                      <mesh filename="package://hsr_meshes/meshes/wrist_v0/wrist_roll.stl" />
+                    </xacro:unless>
+                    <xacro:if value="${g_use_obj_for_collision}">
+                      <mesh filename="package://hsr_meshes/meshes/wrist_v0/wrist_roll.collision.obj" />
+                    </xacro:if>
                 </geometry>
             </collision>
