Commit message: colour for bullet world and gripper-tool-frame

File: urdf/arm_v0/arm.urdf.xacro (robot description, xacro)
@@ -54,4 +54,7 @@
                     </xacro:if>
                 </geometry>
+                <material name="body_main">
+                  <color rgba="0.2 0.2 0.2 1"/>
+                </material>
             </visual>
             <collision>
@@ -85,4 +88,7 @@
                     </xacro:if>
                 </geometry>
+                <material name="body_main">
+                  <color rgba="0.2 0.2 0.2 1"/>
+                </material>
             </visual>
             <collision>
@@ -115,5 +121,9 @@
                         <mesh filename="package://hsr_meshes/meshes/arm_v0/arm_roll_light.obj" />
                     </xacro:if>
+                    	<box size="0.01 0.01 0.01"/>
                 </geometry>
+                <material name="body_main">
+                  <color rgba="0.2 0.2 0.2 1"/>
+                </material>
             </visual>
             <collision>

File: urdf/base_v2/base.urdf.xacro (robot description, xacro)
@@ -58,5 +58,7 @@
                     <cylinder radius="${drive_wheel_radius}" length="${drive_wheel_width}" />
                 </geometry>
-                <material name="wheel" />
+                <material name="wheel">
+                  <color rgba="0.2 0.2 0.2 1.0"/>
+                </material>
             </visual>
             <collision>
@@ -114,5 +116,7 @@
                     <sphere radius="${passive_wheel_radius}" />
                 </geometry>
-                <material name="wheel" />
+                <material name="wheel">
+                  <color rgba="0.2 0.2 0.2 1.0"/>
+                </material>
             </visual>
             <collision>
@@ -151,4 +155,7 @@
                     </xacro:if>
                 </geometry>
+                <material name="body_sub">
+                  <color rgba="0.3333 0.3333 0.3333 1.0"/>
+                </material>
             </visual>
             <visual>
@@ -171,4 +178,7 @@
                     </xacro:if>
                 </geometry>
+                <material name="body_sub">
+                  <color rgba="0.3333 0.3333 0.3333 1.0"/>
+                </material>
             </visual>
             <collision>

File: urdf/hand_v0/hand.urdf.xacro (robot description, xacro)
@@ -89,4 +89,10 @@
             <dynamics damping="1.0"/>
         </joint>
+         <joint name="gripper_tool_joint" type="fixed">
+         <origin rpy="0.0 0.0 -80.14159265359" xyz="0.012 0.0 0.075"/>
+         <parent link="${prefix}_palm_link" />
+          <child link="gripper_tool_frame"/>
+        </joint>
+        <link name="gripper_tool_frame"/>
         <!-- dummy link -->
         <xacro:hsrb_gripper_dummy_link name="${prefix}_motor_dummy_link" />

File: urdf/head_v2/head.urdf.xacro (robot description, xacro)
@@ -57,4 +57,7 @@
                     </xacro:if>
                 </geometry>
+                <material name="tablet">
+                  <color rgba="0.1 0.1 0.2 1.0"/>
+                </material>
             </visual>
             <collision>
@@ -88,4 +91,7 @@
                     </xacro:if>
                 </geometry>
+                <material name="tablet">
+                  <color rgba="0.1 0.1 0.2 1.0"/>
+                </material>
             </visual>
             <visual>
