Commit message: Fixed deprecated xacro syntax

File: urdf/arm_v0/arm.transmission.xacro (robot description, xacro)
@@ -27,7 +27,7 @@
 <robot xmlns:xacro="http://ros.org/wiki/xacro">
     <xacro:macro name="hsrb_arm_transmission" params="prefix">
-        <hsrb_position_joint_transmission joint="${prefix}_lift_joint" reduction="1"/>
-        <hsrb_position_joint_transmission joint="${prefix}_flex_joint" reduction="1"/>
-        <hsrb_position_joint_transmission joint="${prefix}_roll_joint" reduction="1"/>
+        <xacro:hsrb_position_joint_transmission joint="${prefix}_lift_joint" reduction="1"/>
+        <xacro:hsrb_position_joint_transmission joint="${prefix}_flex_joint" reduction="1"/>
+        <xacro:hsrb_position_joint_transmission joint="${prefix}_roll_joint" reduction="1"/>
     </xacro:macro>
 </robot>

File: urdf/base_v2/base.transmission.xacro (robot description, xacro)
@@ -27,7 +27,7 @@
 <robot xmlns:xacro="http://ros.org/wiki/xacro">
     <xacro:macro name="hsrb_base_transmission" params="prefix">
-        <hsrb_velocity_joint_transmission joint="${prefix}_r_drive_wheel_joint" reduction="1"/>
-        <hsrb_velocity_joint_transmission joint="${prefix}_l_drive_wheel_joint" reduction="1"/>
-        <hsrb_position_joint_transmission joint="${prefix}_roll_joint" reduction="1"/>
+        <xacro:hsrb_velocity_joint_transmission joint="${prefix}_r_drive_wheel_joint" reduction="1"/>
+        <xacro:hsrb_velocity_joint_transmission joint="${prefix}_l_drive_wheel_joint" reduction="1"/>
+        <xacro:hsrb_position_joint_transmission joint="${prefix}_roll_joint" reduction="1"/>
     </xacro:macro>
 </robot>

File: urdf/common.xacro (robot description, xacro)
@@ -27,5 +27,5 @@
 <robot xmlns:xacro="http://www.ros.org/wiki.xacro">
   <xacro:arg name="implicit_damping" default="false" />
-  <macro name="hsrb_position_joint_transmission" params="joint reduction">
+  <xacro:macro name="hsrb_position_joint_transmission" params="joint reduction">
      <transmission name="${joint}_transmission">
        <type>transmission_interface/SimpleTransmission</type>
@@ -38,6 +38,6 @@
        </actuator>
      </transmission>
-  </macro>
-  <macro name="hsrb_effort_joint_transmission" params="joint reduction">
+  </xacro:macro>
+  <xacro:macro name="hsrb_effort_joint_transmission" params="joint reduction">
      <transmission name="${joint}_transmission">
        <type>transmission_interface/SimpleTransmission</type>
@@ -50,6 +50,6 @@
        </actuator>
      </transmission>
-  </macro>
-  <macro name="hsrb_velocity_joint_transmission" params="joint reduction">
+  </xacro:macro>
+  <xacro:macro name="hsrb_velocity_joint_transmission" params="joint reduction">
       <transmission name="${prefix}_transmission">
           <type>transmission_interface/SimpleTransmission</type>
@@ -62,6 +62,6 @@
           </actuator>
       </transmission>
-  </macro>
-  <macro name="gazebo_link" params="name gravity collide friction">
+  </xacro:macro>
+  <xacro:macro name="gazebo_link" params="name gravity collide friction">
     <gazebo reference="${name}">
       <selfCollide>${collide}</selfCollide>
@@ -70,6 +70,6 @@
       <mu2>${friction}</mu2>
     </gazebo>
-  </macro>
-  <macro name="gazebo_link_flat_black" params="name gravity collide friction">
+  </xacro:macro>
+  <xacro:macro name="gazebo_link_flat_black" params="name gravity collide friction">
     <gazebo reference="${name}">
       <selfCollide>${collide}</selfCollide>
@@ -79,6 +79,6 @@
       <material value="Gazebo/FlatBlack"/>
     </gazebo>
-  </macro>
-  <macro name="gazebo_link_caster" params="name">
+  </xacro:macro>
+  <xacro:macro name="gazebo_link_caster" params="name">
     <gazebo reference="${name}">
       <selfCollide>false</selfCollide>
@@ -89,6 +89,6 @@
       <material value="Gazebo/FlatBlack"/>
     </gazebo>
-  </macro>
-  <macro name="gazebo_link_rubber" params="name">
+  </xacro:macro>
+  <xacro:macro name="gazebo_link_rubber" params="name">
     <gazebo reference="${name}">
       <selfCollide>false</selfCollide>
@@ -104,6 +104,6 @@
       <material value="Gazebo/FlatBlack"/>
     </gazebo>
-  </macro>
-  <macro name="gazebo_joint" params="name">
+  </xacro:macro>
+  <xacro:macro name="gazebo_joint" params="name">
     <gazebo reference="${name}">
       <xacro:if value="$(arg implicit_damping)">
@@ -111,8 +111,8 @@
       </xacro:if>
     </gazebo>
-  </macro>
-  <macro name="gazebo_joint_mimic" params="name">
+  </xacro:macro>
+  <xacro:macro name="gazebo_joint_mimic" params="name">
     <gazebo reference="${name}">
     </gazebo>
-  </macro>
+  </xacro:macro>
 </robot>

File: urdf/hand_v0/hand.transmission.xacro (robot description, xacro)
@@ -27,7 +27,7 @@
 <robot xmlns:xacro="http://www.ros.org/wiki.xacro">
     <xacro:macro name="hsrb_hand_transmission" params="prefix">
-        <hsrb_effort_joint_transmission joint="${prefix}_motor_joint" reduction="1"/>
-        <hsrb_effort_joint_transmission joint="${prefix}_l_spring_proximal_joint" reduction="1"/>
-        <hsrb_effort_joint_transmission joint="${prefix}_r_spring_proximal_joint" reduction="1"/>
+        <xacro:hsrb_effort_joint_transmission joint="${prefix}_motor_joint" reduction="1"/>
+        <xacro:hsrb_effort_joint_transmission joint="${prefix}_l_spring_proximal_joint" reduction="1"/>
+        <xacro:hsrb_effort_joint_transmission joint="${prefix}_r_spring_proximal_joint" reduction="1"/>
     </xacro:macro>
 </robot>

File: urdf/head_v2/head.transmission.xacro (robot description, xacro)
@@ -27,6 +27,6 @@
 <robot xmlns:xacro="http://ros.org/wiki/xacro">
     <xacro:macro name="hsrb_head_transmission" params="prefix">
-        <hsrb_position_joint_transmission joint="${prefix}_pan_joint" reduction="1"/>
-        <hsrb_position_joint_transmission joint="${prefix}_tilt_joint" reduction="1"/>
+        <xacro:hsrb_position_joint_transmission joint="${prefix}_pan_joint" reduction="1"/>
+        <xacro:hsrb_position_joint_transmission joint="${prefix}_tilt_joint" reduction="1"/>
     </xacro:macro>
 </robot>

File: urdf/wrist_v0/wrist.transmission.xacro (robot description, xacro)
@@ -27,6 +27,6 @@
 <robot xmlns:xacro="http://ros.org/wiki/xacro">
     <xacro:macro name="hsrb_wrist_transmission" params="prefix">
-        <hsrb_position_joint_transmission joint="${prefix}_flex_joint" reduction="1"/>
-        <hsrb_position_joint_transmission joint="${prefix}_roll_joint" reduction="1"/>
+        <xacro:hsrb_position_joint_transmission joint="${prefix}_flex_joint" reduction="1"/>
+        <xacro:hsrb_position_joint_transmission joint="${prefix}_roll_joint" reduction="1"/>
     </xacro:macro>
 </robot>
