Commit message: Fix typo for torso meshes

File: urdf/torso_v0/torso.urdf.xacro (robot description, xacro)
@@ -59,5 +59,5 @@
                 <geometry>
                     <xacro:unless value="${g_use_obj_for_collision}">
-                        <mesh filename="package://hsr_meshes/meshes/torso_v0/torso.std" />
+                        <mesh filename="package://hsr_meshes/meshes/torso_v0/torso.stl" />
                     </xacro:unless>
                     <xacro:if value="${g_use_obj_for_collision}">
