Commit message: Remove globally defined variable pi

File: urdf/common.xacro (robot description, xacro)
@@ -27,5 +27,4 @@
 <robot xmlns:xacro="http://www.ros.org/wiki.xacro">
   <xacro:arg name="implicit_damping" default="false" />
-  <xacro:property name="pi" value="3.14159265359"/>
   <macro name="hsrb_position_joint_transmission" params="joint reduction">
      <transmission name="${joint}_transmission">
